File: GigaTOLT.kicad_pcb (KiCad board)
At the start: 4 copper layers, 100 x 79.9 mm, 171 parts, among them J1 MOTOR SENSORS, J2 CAN, J3 UART / I2C, J301 GigaControl_Card_Interface, J4 SPI / EXPANSION, J401 GigaPower_Card_Interface, J5 USB / SERVO, J6 Conn_02x03_Counter_Clockwise, Q1 IPTC034N15NM6ATMA1, Q10 IPTC034N15NM6ATMA1, Q2 IPTC034N15NM6ATMA1, Q23 IPTC034N15NM6ATMA1, Q24 IPTC034N15NM6ATMA1, Q25 IPTC034N15NM6ATMA1, Q3 IPTC034N15NM6ATMA1, Q5 IPTC034N15NM6ATMA1, Q6 IPTC034N15NM6ATMA1, Q7 IPTC034N15NM6ATMA1, Q8 IPTC034N15NM6ATMA1, Q9 IPTC034N15NM6ATMA1, U11 ACS37030, U13 ACS37030, U15 ACS37030, U6 2EDF7275K, U7 2EDF7275K, U8 2EDF7275K

Commit message: initial
Parts:
- added NT1: NetTie_2, NetTie:NetTie-2_SMD_Pad2.0mm, F.Cu at (115.1, 110.0)
- moved R23 16.9 mm to (179.2, 129.5), turned to -45 degrees
- moved C27 15.0 mm to (181.0, 131.2), turned to -45 degrees
- moved J3 13.5 mm to (161.4, 121.1), turned to 90 degrees
- moved D18 10.3 mm to (154.7, 123.7)
- moved D19 9.62 mm to (154.6, 121.3)
- moved R64 9.19 mm to (119.2, 116.8), turned to -90 degrees
- moved R40 9.05 mm to (151.4, 123.5)
- moved J5 6.75 mm to (174.8, 121.1), turned to 90 degrees
- moved J2 6.70 mm to (167.9, 121.1), turned to 90 degrees
- moved R63 6.09 mm to (117.3, 116.8), turned to -90 degrees
- moved JP3 5.11 mm to (196.8, 119.9), turned to -90 degrees
- moved J6 3.70 mm to (199.4, 123.1)
- moved J1 3.70 mm to (192.1, 121.4), turned to 90 degrees
- moved R62 3.14 mm to (115.5, 116.8), turned to -90 degrees
- moved R69 2.40 mm to (142.0, 106.4), turned to 90 degrees
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Connections:
- J301 pad J33_14: IN-CANH -> IN-CANL
- J301 pad J33_16: IN-CANL -> IN-CANH
Routing:
- net GND: track 262.6 -> 104.0 mm, vias 100 -> 69
- net +3.3V: track 171.7 -> 312.6 mm, vias 5 -> 12
- net POWER-STAGE-LOCKOUT: track 0.00 -> 122.1 mm, vias 0 -> 5
- net +12V: track 91.3 -> 178.5 mm, vias 1 -> 3
- net +5V: track 0.00 -> 67.7 mm, vias 0 -> 3
- net IN-V: track 0.00 -> 62.9 mm
- net L1: track 0.00 -> 61.7 mm
- net H1: track 0.00 -> 61.6 mm
- net IN-CANH: track 0.00 -> 44.5 mm, vias 0 -> 1
- net I2C2-SDA/USART3-RX: track 0.00 -> 43.0 mm, vias 0 -> 2
- net MOSTEMP3: track 18.5 -> 61.3 mm, vias 0 -> 2
- net Net-(Q9-G): track 43.8 -> 7.49 mm
- net MOSTEMP2: track 23.5 -> 58.7 mm, vias 0 -> 3
- net CURR3-FILTERED: track 2.22 -> 36.8 mm
- net CURR1-FILTERED: track 27.3 -> 60.3 mm
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