File: GigaTOLT.kicad_pcb (KiCad board)
At the start: 4 copper layers, 100 x 79.9 mm, 172 parts, among them J1 MOTOR SENSORS, J2 CAN, J3 UART / I2C, J301 GigaControl_Card_Interface, J4 SPI / EXPANSION, J401 GigaPower_Card_Interface, J5 USB / SERVO, J6 Conn_02x03_Counter_Clockwise, Q1 IPTC034N15NM6ATMA1, Q10 IPTC034N15NM6ATMA1, Q2 IPTC034N15NM6ATMA1, Q23 IPTC034N15NM6ATMA1, Q24 IPTC034N15NM6ATMA1, Q25 IPTC034N15NM6ATMA1, Q3 IPTC034N15NM6ATMA1, Q5 IPTC034N15NM6ATMA1, Q6 IPTC034N15NM6ATMA1, Q7 IPTC034N15NM6ATMA1, Q8 IPTC034N15NM6ATMA1, Q9 IPTC034N15NM6ATMA1, U11 ACS37030, U13 ACS37030, U15 ACS37030, U6 2EDF7275K, U7 2EDF7275K, U8 2EDF7275K

Commit message: initial
Parts:
- removed NT1: NetTie_2, NetTie:NetTie-2_SMD_Pad2.0mm
- C109, C139, C79: moved to F.Cu
- moved H7 4.10 mm to (127.1, 63.4)
- moved H8 4.10 mm to (156.0, 63.3)
- moved H9 4.10 mm to (184.9, 63.3)
- moved C109 3.40 mm to (167.6, 59.9), turned to 0 degrees
- moved C139 3.40 mm to (196.5, 59.9), turned to 0 degrees
- moved C79 3.40 mm to (138.7, 60.0), turned to 0 degrees
- moved H6 0.70 mm to (206.5, 128.6)
- moved D18 0.50 mm to (154.7, 123.2)
- moved R40 0.30 mm to (151.4, 123.2), turned to 180 degrees
- moved H1 0.20 mm to (206.5, 97.4)
- moved H10 0.20 mm to (204.5, 71.1)
- moved C128 0.10 mm to (202.9, 84.7)
- moved C68 0.10 mm to (145.1, 84.8)
- moved C98 0.10 mm to (174.0, 84.7)
- moved TH1 0.10 mm to (144.2, 87.1)
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Routing:
- net GND: track 104.0 -> 214.3 mm, vias 69 -> 143
- net +BATT: track 175.7 -> 210.8 mm
- net +3.3V: track 312.6 -> 302.0 mm, vias 12 -> 11
- net +12V: track 178.5 -> 171.1 mm
- net /DriverSocketPhase3/VSW: track 292.5 -> 298.6 mm
- net I2C2-SDA/USART3-RX: track 43.0 -> 39.3 mm
- net /DriverSocketPhase2/VSW: track 292.5 -> 295.9 mm
- net I2C2-SCL/USART3-TX: track 43.8 -> 40.9 mm
- net Net-(Q9-G): track 7.49 -> 9.95 mm
- net L1: track 61.7 -> 59.2 mm
- net H1: track 61.6 -> 59.3 mm
- net IN-V: track 62.9 -> 65.0 mm
- net POWER-STAGE-DISABLE: track 21.6 -> 23.7 mm
- net Net-(R61-Pad2): track 0.00 -> 1.91 mm
- net Net-(R62-Pad2): track 0.00 -> 1.80 mm
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Other:
- board text added: "GigaESC TOLT - v2.0.0 By Kaminaris"
- board text removed: "GigaESC TOLT - v1.0.0 By Kaminaris"
