File: GigaTOLT.kicad_pcb (KiCad board)
At the start: 4 copper layers, 100 x 79.9 mm, 171 parts, among them J1 MOTOR SENSORS, J2 CAN, J3 UART / I2C, J301 GigaControl_Card_Interface, J4 SPI / EXPANSION, J401 GigaPower_Card_Interface, J5 USB / SERVO, J6 Conn_02x03_Counter_Clockwise, Q1 IPTC034N15NM6ATMA1, Q10 IPTC034N15NM6ATMA1, Q2 IPTC034N15NM6ATMA1, Q23 IPTC034N15NM6ATMA1, Q24 IPTC034N15NM6ATMA1, Q25 IPTC034N15NM6ATMA1, Q3 IPTC034N15NM6ATMA1, Q5 IPTC034N15NM6ATMA1, Q6 IPTC034N15NM6ATMA1, Q7 IPTC034N15NM6ATMA1, Q8 IPTC034N15NM6ATMA1, Q9 IPTC034N15NM6ATMA1, U11 ACS37030, U13 ACS37030, U15 ACS37030, U6 2EDF7275K, U7 2EDF7275K, U8 2EDF7275K

Commit message: clearance
Parts:
- added C51: 100n, Capacitor_SMD:C_0805_2012Metric, F.Cu at (139.4, 84.4)
- added C52: 3.3u, Capacitor_SMD:C_2220_5750Metric, F.Cu at (121.8, 88.4)
- added C53: 100n, Capacitor_SMD:C_0805_2012Metric, F.Cu at (123.0, 84.4)
- added C56: 100n, Capacitor_SMD:C_0805_2012Metric, F.Cu at (168.3, 84.4)
- added C57: 3.3u, Capacitor_SMD:C_2220_5750Metric, F.Cu at (150.7, 88.4)
- added C59: 100n, Capacitor_SMD:C_0805_2012Metric, F.Cu at (151.9, 84.4)
- added C60: 100n, Capacitor_SMD:C_0805_2012Metric, F.Cu at (197.2, 84.4)
- added C61: 3.3u, Capacitor_SMD:C_2220_5750Metric, F.Cu at (179.6, 88.4)
- added C65: 3.3u, Capacitor_SMD:C_2220_5750Metric, F.Cu at (140.6, 88.4)
- added C66: 3.3u, Capacitor_SMD:C_2220_5750Metric, F.Cu at (169.5, 88.4)
- added C67: 3.3u, Capacitor_SMD:C_2220_5750Metric, F.Cu at (198.4, 88.4)
- added C69: 100n, Capacitor_SMD:C_0805_2012Metric, F.Cu at (180.8, 84.4)
- moved C46 7.44 mm to (151.9, 98.3), turned to 180 degrees
- moved C47 7.44 mm to (180.8, 98.3), turned to 180 degrees
- moved C58 7.44 mm to (197.2, 98.3), turned to 0 degrees
- moved C54 7.44 mm to (168.3, 98.3), turned to 0 degrees
- moved C45 7.36 mm to (123.0, 98.3), turned to 180 degrees
- moved C50 7.36 mm to (139.4, 98.3), turned to 0 degrees
- moved R74 2.20 mm to (129.2, 80.7)
- moved TH1 2.20 mm to (144.3, 84.9)
- moved R68 2.20 mm to (133.2, 80.7)
- moved C68 2.20 mm to (145.1, 82.6)
- moved R67 2.20 mm to (143.6, 82.6)
- moved U11 2.20 mm to (138.9, 80.7)
- moved C71 2.20 mm to (143.5, 79.9)
- moved R75 2.10 mm to (158.1, 80.7)
- moved R76 2.10 mm to (187.0, 80.7)
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Routing:
- net GND: track 214.3 -> 221.2 mm, vias 143 -> 185
- net +3.3V: track 302.0 -> 308.2 mm
- net +BATT: track 210.8 -> 215.6 mm, vias 56 -> 74
- net MOSTEMP1: track 82.1 -> 86.9 mm
- net MOSTEMP3: track 59.7 -> 64.4 mm
- net MOSTEMP2: track 57.7 -> 62.3 mm
- net Net-(Q9-G): track 9.95 -> 7.49 mm
- net Net-(U11-VOUT): track 30.0 -> 32.2 mm
- net Net-(U13-VOUT): track 30.0 -> 32.2 mm
- net Net-(U15-VOUT): track 30.0 -> 32.2 mm
- net +12V: track 171.1 -> 169.0 mm
- net Net-(D9-K): track 5.78 -> 3.72 mm
- net Net-(D8-K): track 5.78 -> 3.72 mm
- net Net-(D7-K): track 5.78 -> 3.72 mm
- net /DriverSocketPhase3/VSW: track 298.6 -> 297.2 mm, vias 42 -> 68
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- added copper zone on In1.Cu, net +BATT
- added copper zone on In2.Cu, net +BATT
