File: DriverSocket.kicad_sch (KiCad schematic)
At the start: 31 parts, among them U11 ACS37030, U6 2EDF7275K

Commit message: initial
Parts:
- C79: footprint GigaTOLTLibrary:CapacitorD18x32 -> Capacitor_THT:CP_Radial_D18.0mm_P7.50mm
Changed lines of the file:
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@@
 			)
 		)
-		(property "Footprint" "GigaTOLTLibrary:CapacitorD18x32"
+		(property "Footprint" "Capacitor_THT:CP_Radial_D18.0mm_P7.50mm"
 			(at 230.8352 72.39 0)
 			(hide yes)

Commit message: clearance
Parts:
- added C51, C53: 100n, Capacitor_SMD:C_0805_2012Metric, symbol Device:C
- added C52, C65: 3.3u, Capacitor_SMD:C_2220_5750Metric, symbol Device:C
- C48, C62: MPN C5156756 -> C22370027
- C79: footprint Capacitor_THT:CP_Radial_D18.0mm_P7.50mm -> GigaTOLTLibrary:CapacitorD18x32
Connections:
- net +BATT: now also C51.1, C52.1, C53.1, C65.1
- net GND: now also C51.2, C52.2, C53.2, C65.2
Other:
- moved on the sheet: C45, C48, C50, C62
