File: FetPair.kicad_sch (KiCad schematic)
At the start: 8 parts, among them Q1 IPTC034N15NM6ATMA1, Q7 IPTC034N15NM6ATMA1

Commit message: clearance
Parts:
- C5, C6: MPN (none) -> C53987
- L11, L5: MPN (none) -> C113019
Connections:
- net +BATT: no longer Q1.17 (D_9)
- net PHASE: no longer Q7.17 (D_9)
Changed lines of the file:
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@@
+			)
+		)
+		(property "MPN" "C113019"
+			(at 104.14 109.22 0)
+			(hide yes)
+			(show_name no)
+			(do_not_autoplace no)
+			(effects
+				(font
+					(size 1.27 1.27)
+				)
 			)
 		)
@@
 			)
 		)
+		(property "MPN" "C53987"
+			(at 128.27 119.3799 0)
+			(hide yes)
+			(show_name no)
+			(do_not_autoplace no)
+			(effects
+				(font
+					(size 1.27 1.27)
+				)
+			)
+		)
 		(property "Footprint" "Capacitor_SMD:C_0603_1608Metric"
 			(at 125.4252 121.92 0)
@@
 		(pin "16"
 		)
-		(pin "17"
-		)
 		(instances
 			(project "GigaTOLT"
@@
 		(pin "16"
 		)
-		(pin "17"
-		)
 		(pin "12"
 		)
@@
 			)
 		)
+		(property "MPN" "C113019"
+			(at 105.41 83.82 0)
+			(hide yes)
+			(show_name no)
+			(do_not_autoplace no)
+			(effects
+				(font
+					(size 1.27 1.27)
+				)
+			)
+		)
 		(property "Footprint" "Inductor_SMD:L_0603_1608Metric"
 			(at 105.41 86.36 0)
@@
 			)
 		)
+		(property "MPN" "C53987"
+			(at 128.27 93.9799 0)
+			(hide yes)
+			(show_name no)
+			(do_not_autoplace no)
+			(effects
+				(font
+					(size 1.27 1.27)
+				)
+			)
+		)
